File: pcb/futaba-pcb/futaba-pcb.kicad_pcb (KiCad board)
At the start: 2 copper layers, 324.5 x 114.9 mm, 105 parts, among them J1 Conn_01x06, SW1 SW_Push, SW10 SW_Push, SW11 SW_Push, SW12 SW_Push, SW13 SW_Push, SW14 SW_Push, SW15 SW_Push, SW16 SW_Push, SW17 SW_Push, SW18 SW_Push, SW2 SW_Push, SW20 SW_Push, SW21 SW_Push, SW22 SW_Push, SW23 SW_Push, SW24 SW_Push, SW25 SW_Push, SW26 SW_Push, SW27 SW_Push, SW28 SW_Push, SW29 SW_Push, SW3 SW_Push, SW30 SW_Push, SW31 SW_Push, SW32 SW_Push, SW33 SW_Push, SW34 SW_Push, SW35 SW_Push, SW36 SW_Push, SW37 SW_Push, SW38 SW_Push, SW39 SW_Push, SW4 SW_Push, SW40 SW_Push, SW41 SW_Push, SW42 SW_Push, SW44 SW_Push, SW45 SW_Push, SW46 SW_Push, SW47 SW_Push, SW48 SW_Push, SW49 SW_Push, SW5 SW_Push, SW50 SW_Push, SW51 SW_Push, SW6 SW_Push, SW7 SW_Push, SW8 SW_Push, SW9 SW_Push, U1 RP2040-Zero

Commit message: Update pcb data
Parts:
- EC12, MSW1: moved to B.Cu
- SW1, SW2, SW22, SW23, SW24, SW3, SW4, SW5, SW6: footprint keyboard:Choc_Socket -> keyboard:Choc_Socket-flex-drill_top
- SW10, SW11, SW12, SW13, SW14, SW15, SW16, SW17, SW18, SW7, SW8, SW9: footprint keyboard:Choc_Socket -> keyboard:Choc_Socket-flex-drill
- SW20, SW21: footprint keyboard:Choc_Socket -> keyboard:Choc_Socket-flex-drill_bottom
- SW25, SW26, SW27, SW28, SW29, SW30, SW31, SW32, SW33, SW34, SW35, SW36, SW37, SW38, SW39, SW40, SW41, SW42, SW44, SW45, SW46, SW47, SW48: footprint keyboard:Choc_Socket -> keyboard:Choc_Socket-flex-drill_2
- moved D19 35.1 mm to (210.7, 136.7), turned to -90 degrees
- moved MSW1 14.1 mm to (213.3, 141.1), turned to 180 degrees
- moved J1 5.96 mm to (216.2, 128.8)
- moved EC12 5.69 mm to (200.9, 161.7)
- moved U1 5.60 mm to (198.4, 132.7)
- moved R2 5.07 mm to (219.9, 131.5)
- moved R1 5.07 mm to (217.0, 131.5)
- moved D37 2.70 mm to (50.2, 115.8)
- moved D31 2.42 mm to (53.9, 96.8)
- moved D48 2.38 mm to (158.5, 158.3)
- moved D35 2.36 mm to (131.1, 97.5)
- moved D28 2.34 mm to (117.5, 68.5)
- moved D36 2.34 mm to (149.1, 105.1)
- moved D29 2.33 mm to (134.8, 78.8)
- moved D25 2.31 mm to (57.5, 78.2)
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Connections:
- U1 pad 10: /RR4 -> /LR1
- U1 pad 11: /RR1 -> /LR4
- U1 pad 12: /RR2 -> unconnected-(U1-GP12-Pad12)
- U1 pad 13: /RR3 -> /RotaryA
- U1 pad 14: /SDA -> /RotaryB
- U1 pad 15: /SCL -> /RR4
- U1 pad 2: /C6 -> /SDA
- U1 pad 26: /CR1 -> /RR1
- U1 pad 27: unconnected-(U1-GP27-Pad27) -> /RR2
- U1 pad 28: /RotaryB -> /RR3
- U1 pad 29: /RotaryA -> /CR1
- U1 pad 3: /C1 -> /SCL
- U1 pad 4: /C2 -> /C6
- U1 pad 6: /LR3 -> /C1
- U1 pad 7: /LR2 -> /C2
- U1 pad 8: /LR1 -> /LR2
- U1 pad 9: /LR4 -> /LR3
Routing:
- net /LR3: track 329.6 -> 684.8 mm
- net /LR2: track 353.0 -> 523.8 mm
- net /RR3: track 332.8 -> 412.8 mm
- net /RR2: track 356.2 -> 435.9 mm
- net /RR1: track 381.1 -> 457.2 mm
- net /RR4: track 237.2 -> 308.5 mm
- net /LR4: track 251.6 -> 280.8 mm
- net /SDA: track 47.0 -> 20.7 mm
- net Net-(D19-A): track 27.7 -> 2.67 mm, vias 1 -> 0
- net /SCL: track 46.7 -> 22.1 mm
- net /CR1: track 358.8 -> 383.1 mm
- net /RotaryB: track 59.3 -> 37.8 mm, vias 2 -> 0
- net /C4: track 801.0 -> 780.1 mm, vias 18 -> 19
- net /LR1: track 378.1 -> 393.6 mm
- net +3.3V: track 37.3 -> 50.8 mm
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Other:
- outline, holes or cut-outs redrawn
