File: pcb/futaba-pcb/futaba-pcb.kicad_sch (KiCad schematic)
At the start: 105 parts, among them J1 Conn_01x06, SW1 SW_Push, SW10 SW_Push, SW11 SW_Push, SW12 SW_Push, SW13 SW_Push, SW14 SW_Push, SW15 SW_Push, SW16 SW_Push, SW17 SW_Push, SW18 SW_Push, SW2 SW_Push, SW20 SW_Push, SW21 SW_Push, SW22 SW_Push, SW23 SW_Push, SW24 SW_Push, SW25 SW_Push, SW26 SW_Push, SW27 SW_Push, SW28 SW_Push, SW29 SW_Push, SW3 SW_Push, SW30 SW_Push, SW31 SW_Push, SW32 SW_Push, SW33 SW_Push, SW34 SW_Push, SW35 SW_Push, SW36 SW_Push, SW37 SW_Push, SW38 SW_Push, SW39 SW_Push, SW4 SW_Push, SW40 SW_Push, SW41 SW_Push, SW42 SW_Push, SW44 SW_Push, SW45 SW_Push, SW46 SW_Push, SW47 SW_Push, SW48 SW_Push, SW49 SW_Push, SW5 SW_Push, SW50 SW_Push, SW51 SW_Push, SW6 SW_Push, SW7 SW_Push, SW8 SW_Push, SW9 SW_Push, U1 RP2040-Zero

Commit message: Update pcb data
Parts:
- SW1, SW2, SW22, SW23, SW24, SW3, SW4, SW5, SW6: footprint keyboard:Choc_Socket -> keyboard:Choc_Socket-flex-drill_top
- SW10, SW11, SW12, SW13, SW14, SW15, SW16, SW17, SW18, SW7, SW8, SW9: footprint keyboard:Choc_Socket -> keyboard:Choc_Socket-flex-drill
- SW20, SW21: footprint keyboard:Choc_Socket -> keyboard:Choc_Socket-flex-drill_bottom
- SW25, SW26, SW27, SW28, SW29, SW30, SW31, SW32, SW33, SW34, SW35, SW36, SW37, SW38, SW39, SW40, SW41, SW42, SW44, SW45, SW46, SW47, SW48: footprint keyboard:Choc_Socket -> keyboard:Choc_Socket-flex-drill_2
Connections:
- net C1: now also U1.6 (GP6); no longer U1.3 (GP3)
- net C2: now also U1.7 (GP7); no longer U1.4 (GP4)
- net C6: now also U1.4 (GP4); no longer U1.2 (GP2)
- net CR1: now also U1.29 (GP29); no longer U1.26 (GP26)
- net LR1: now also U1.10 (GP10); no longer U1.8 (GP8)
- net LR2: now also U1.8 (GP8); no longer U1.7 (GP7)
- net LR3: now also U1.9 (GP9); no longer U1.6 (GP6)
- net LR4: now also U1.11 (GP11); no longer U1.9 (GP9)
- net RR1: now also U1.26 (GP26); no longer U1.11 (GP11)
- net RR2: now also U1.27 (GP27); no longer U1.12 (GP12)
- net RR3: now also U1.28 (GP28); no longer U1.13 (GP13)
- net RR4: now also U1.15 (GP15); no longer U1.10 (GP10)
- net RotaryA: now also U1.13 (GP13); no longer U1.29 (GP29)
- net RotaryB: now also U1.14 (GP14); no longer U1.28 (GP28)
- net SCL: now also U1.3 (GP3); no longer U1.15 (GP15)
- net SDA: now also U1.2 (GP2); no longer U1.14 (GP14)
Changed lines of the file:
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@@
 	)
 	(no_connect
-		(at 243.84 74.93)
+		(at 257.81 86.36)
 	)
 	(no_connect
@@
 	)
 	(label "LR2"
-		(at 275.59 80.01 0)
+		(at 275.59 82.55 0)
 		(fields_autoplaced yes)
 		(effects
@@
 	)
 	(label "RR3"
-		(at 255.27 86.36 270)
+		(at 243.84 72.39 180)
 		(fields_autoplaced yes)
 		(effects
@@
 	)
 	(label "SDA"
-		(at 243.84 82.55 180)
+		(at 275.59 67.31 0)
 		(fields_autoplaced yes)
 		(effects
@@
 				(size 1.27 1.27)
 			)
-			(justify right bottom)
+			(justify left bottom)
 		)
 	)
@@
 	)
 	(label "LR4"
-		(at 265.43 86.36 270)
+		(at 260.35 86.36 270)
 		(fields_autoplaced yes)
 		(effects
@@
 	)
 	(label "CR1"
-		(at 243.84 77.47 180)
+		(at 243.84 69.85 180)
 		(fields_autoplaced yes)
 		(effects
@@
 	)
 	(label "RR1"
-		(at 260.35 86.36 270)
+		(at 243.84 77.47 180)
 		(fields_autoplaced yes)
 		(effects
@@
 	)
 	(label "RotaryB"
-		(at 243.84 72.39 180)
+		(at 243.84 82.55 180)
 		(fields_autoplaced yes)
 		(effects
@@
 	)
 	(label "RR2"
-		(at 257.81 86.36 270)
+		(at 243.84 74.93 180)
 		(fields_autoplaced yes)
 		(effects
@@
 	)
 	(label "RotaryA"
-		(at 243.84 69.85 180)
+		(at 255.27 86.36 270)
 		(fields_autoplaced yes)
 		(effects
@@
 	)
 	(label "C2"
-		(at 275.59 72.39 0)
+		(at 275.59 80.01 0)
 		(fields_autoplaced yes)
 		(effects
@@
 	)
 	(label "LR3"
-		(at 275.59 77.47 0)
+		(at 265.43 86.36 270)
 		(fields_autoplaced yes)
 		(effects
@@
 				(size 1.27 1.27)
 			)
-			(justify left bottom)
+			(justify right bottom)
 		)
 	)
 	(label "C1"
-		(at 275.59 69.85 0)
+		(at 275.59 77.47 0)
 		(fields_autoplaced yes)
 		(effects
@@
 	)
 	(label "LR1"
-		(at 275.59 82.55 0)
+		(at 262.89 86.36 270)
 		(fields_autoplaced yes)
 		(effects
@@
 				(size 1.27 1.27)
 			)
-			(justify left bottom)
+			(justify right bottom)
 		)
 	)
@@
 	)
 	(label "C6"
-		(at 275.59 67.31 0)
+		(at 275.59 72.39 0)
 		(fields_autoplaced yes)
 		(effects
@@
 	)
 	(label "SCL"
-		(at 243.84 80.01 180)
+		(at 275.59 69.85 0)
 		(fields_autoplaced yes)
 		(effects
@@
 				(size 1.27 1.27)
 			)
-			(justify right bottom)
+			(justify left bottom)
 		)
 	)
@@
 	)
 	(label "RR4"
-		(at 262.89 86.36 270)
+		(at 243.84 80.01 180)
 		(fields_autoplaced yes)
 		(effects
@@
 			)
 		)
-		(property "Footprint" "keyboard:Choc_Socket"
+		(property "Footprint" "keyboard:Choc_Socket-flex-drill_top"
 			(at 166.37 116.84 0)
 			(effects
@@
 			)
 		)
-		(property "Footprint" "keyboard:Choc_Socket"
+		(property "Footprint" "keyboard:Choc_Socket-flex-drill_2"
 			(at 118.11 193.04 0)
 			(effects
@@
 			)
 		)
-		(property "Footprint" "keyboard:Choc_Socket"
+		(property "Footprint" "keyboard:Choc_Socket-flex-drill_2"
 			(at 93.98 135.89 0)
 			(effects
@@
 			)
 		)
-		(property "Footprint" "keyboard:Choc_Socket"
+		(property "Footprint" "keyboard:Choc_Socket-flex-drill_2"
 			(at 93.98 154.94 0)
 			(effects
@@
 			)
 		)
-		(property "Footprint" "keyboard:Choc_Socket"
+		(property "Footprint" "keyboard:Choc_Socket-flex-drill"
 			(at 118.11 74.93 0)
 			(effects
@@
 			)
 		)
-		(property "Footprint" "keyboard:Choc_Socket"
+		(property "Footprint" "keyboard:Choc_Socket-flex-drill_2"
 			(at 166.37 173.99 0)
 			(effects
@@
 			)
 		)
-		(property "Footprint" "keyboard:Choc_Socket"
+		(property "Footprint" "keyboard:Choc_Socket-flex-drill_top"
 			(at 166.37 52.07 0)
 			(effects
@@
 			)
 		)
-		(property "Footprint" "keyboard:Choc_Socket"
+		(property "Footprint" "keyboard:Choc_Socket-flex-drill"
 			(at 93.98 96.52 0)
 			(effects
@@
 			)
 		)
-		(property "Footprint" "keyboard:Choc_Socket"
+		(property "Footprint" "keyboard:Choc_Socket-flex-drill_2"
 			(at 142.24 193.04 0)
 			(effects
@@
 			)
 		)
-		(property "Footprint" "keyboard:Choc_Socket"
+		(property "Footprint" "keyboard:Choc_Socket-flex-drill_2"
 			(at 45.72 154.94 0)
 			(effects
@@
 			)
 		)
-		(property "Footprint" "keyboard:Choc_Socket"
+		(property "Footprint" "keyboard:Choc_Socket-flex-drill_2"
 			(at 69.85 173.99 0)
 			(effects
@@
 			)
 		)
-		(property "Footprint" "keyboard:Choc_Socket"
+		(property "Footprint" "keyboard:Choc_Socket-flex-drill_2"
 			(at 45.72 173.99 0)
 			(effects
@@
 			)
 		)
-		(property "Footprint" "keyboard:Choc_Socket"
+		(property "Footprint" "keyboard:Choc_Socket-flex-drill"
 			(at 69.85 74.93 0)
 			(effects
@@
 			)
 		)
-		(property "Footprint" "keyboard:Choc_Socket"
+		(property "Footprint" "keyboard:Choc_Socket-flex-drill_2"
 			(at 142.24 135.89 0)
 			(effects
@@
 			)
 		)
-		(property "Footprint" "keyboard:Choc_Socket"
+		(property "Footprint" "keyboard:Choc_Socket-flex-drill_top"
 			(at 93.98 52.07 0)
 			(effects
@@
 			)
 		)
-		(property "Footprint" "keyboard:Choc_Socket"
+		(property "Footprint" "keyboard:Choc_Socket-flex-drill_2"
 			(at 142.24 173.99 0)
 			(effects
@@
 			)
 		)
-		(property "Footprint" "keyboard:Choc_Socket"
+		(property "Footprint" "keyboard:Choc_Socket-flex-drill_top"
 			(at 69.85 52.07 0)
 			(effects
@@
 			)
 		)
-		(property "Footprint" "keyboard:Choc_Socket"
+		(property "Footprint" "keyboard:Choc_Socket-flex-drill"
 			(at 45.72 96.52 0)
 			(effects
@@
 			)
 		)
-		(property "Footprint" "keyboard:Choc_Socket"
+		(property "Footprint" "keyboard:Choc_Socket-flex-drill_2"
 			(at 142.24 154.94 0)
 			(effects
@@
 			)
 		)
-		(property "Footprint" "keyboard:Choc_Socket"
+		(property "Footprint" "keyboard:Choc_Socket-flex-drill_2"
 			(at 166.37 193.04 0)
 			(effects
@@
 			)
 		)
-		(property "Footprint" "keyboard:Choc_Socket"
+		(property "Footprint" "keyboard:Choc_Socket-flex-drill_2"
 			(at 166.37 154.94 0)
 			(effects
@@
 			)
 		)
-		(property "Footprint" "keyboard:Choc_Socket"
+		(property "Footprint" "keyboard:Choc_Socket-flex-drill_top"
 			(at 142.24 52.07 0)
 			(effects
@@
 			)
 		)
-		(property "Footprint" "keyboard:Choc_Socket"
+		(property "Footprint" "keyboard:Choc_Socket-flex-drill_2"
 			(at 69.85 135.89 0)
 			(effects
@@
 			)
 		)
-		(property "Footprint" "keyboard:Choc_Socket"
+		(property "Footprint" "keyboard:Choc_Socket-flex-drill_2"
 			(at 118.11 173.99 0)
 			(effects
@@
 			)
 		)
-		(property "Footprint" "keyboard:Choc_Socket"
+		(property "Footprint" "keyboard:Choc_Socket-flex-drill_2"
 			(at 45.72 135.89 0)
 			(effects
@@
 			)
 		)
-		(property "Footprint" "keyboard:Choc_Socket"
+		(property "Footprint" "keyboard:Choc_Socket-flex-drill_bottom"
 			(at 69.85 116.84 0)
 			(effects
@@
 			)
 		)
-		(property "Footprint" "keyboard:Choc_Socket"
+		(property "Footprint" "keyboard:Choc_Socket-flex-drill_2"
 			(at 118.11 154.94 0)
 			(effects
@@
 			)
 		)
-		(property "Footprint" "keyboard:Choc_Socket"
+		(property "Footprint" "keyboard:Choc_Socket-flex-drill_2"
 			(at 69.85 154.94 0)
 			(effects
@@
 			)
 		)
-		(property "Footprint" "keyboard:Choc_Socket"
+		(property "Footprint" "keyboard:Choc_Socket-flex-drill"
 			(at 45.72 74.93 0)
 			(effects
@@
 			)
 		)
-		(property "Footprint" "keyboard:Choc_Socket"
+		(property "Footprint" "keyboard:Choc_Socket-flex-drill_top"
 			(at 45.72 52.07 0)
 			(effects
@@
 			)
 		)
-		(property "Footprint" "keyboard:Choc_Socket"
+		(property "Footprint" "keyboard:Choc_Socket-flex-drill_top"
 			(at 142.24 116.84 0)
 			(effects
@@
 			)
 		)
-		(property "Footprint" "keyboard:Choc_Socket"
+		(property "Footprint" "keyboard:Choc_Socket-flex-drill_2"
 			(at 93.98 173.99 0)
 			(effects
@@
 			)
 		)
-		(property "Footprint" "keyboard:Choc_Socket"
+		(property "Footprint" "keyboard:Choc_Socket-flex-drill_2"
 			(at 69.85 193.04 0)
 			(effects
@@
 			)
 		)
-		(property "Footprint" "keyboard:Choc_Socket"
+		(property "Footprint" "keyboard:Choc_Socket-flex-drill"
 			(at 166.37 74.93 0)
 			(effects
@@
 			)
 		)
-		(property "Footprint" "keyboard:Choc_Socket"
+		(property "Footprint" "keyboard:Choc_Socket-flex-drill"
 			(at 118.11 96.52 0)
 			(effects
@@
 			)
 		)
-		(property "Footprint" "keyboard:Choc_Socket"
+		(property "Footprint" "keyboard:Choc_Socket-flex-drill"
 			(at 93.98 74.93 0)
 			(effects
@@
 			)
 		)
-		(property "Footprint" "keyboard:Choc_Socket"
+		(property "Footprint" "keyboard:Choc_Socket-flex-drill_top"
 			(at 118.11 116.84 0)
 			(effects
@@
 			)
 		)
-		(property "Footprint" "keyboard:Choc_Socket"
+		(property "Footprint" "keyboard:Choc_Socket-flex-drill_top"
 			(at 118.11 52.07 0)
 			(effects
@@
 			)
 		)
-		(property "Footprint" "keyboard:Choc_Socket"
+		(property "Footprint" "keyboard:Choc_Socket-flex-drill"
 			(at 142.24 74.93 0)
 			(effects
@@
 			)
 		)
-		(property "Footprint" "keyboard:Choc_Socket"
+		(property "Footprint" "keyboard:Choc_Socket-flex-drill_bottom"
 			(at 93.98 116.84 0)
 			(effects
@@
 			)
 		)
-		(property "Footprint" "keyboard:Choc_Socket"
+		(property "Footprint" "keyboard:Choc_Socket-flex-drill_2"
 			(at 166.37 135.89 0)
 			(effects
@@
 			)
 		)
-		(property "Footprint" "keyboard:Choc_Socket"
+		(property "Footprint" "keyboard:Choc_Socket-flex-drill_2"
 			(at 93.98 193.04 0)
 			(effects
@@
 			)
 		)
-		(property "Footprint" "keyboard:Choc_Socket"
+		(property "Footprint" "keyboard:Choc_Socket-flex-drill"
 			(at 69.85 96.52 0)
 			(effects
@@
 			)
 		)
-		(property "Footprint" "keyboard:Choc_Socket"
+		(property "Footprint" "keyboard:Choc_Socket-flex-drill"
 			(at 166.37 96.52 0)
 			(effects
@@
 			)
 		)
-		(property "Footprint" "keyboard:Choc_Socket"
+		(property "Footprint" "keyboard:Choc_Socket-flex-drill_2"
 			(at 118.11 135.89 0)
 			(effects
@@
 			)
 		)
-		(property "Footprint" "keyboard:Choc_Socket"
+		(property "Footprint" "keyboard:Choc_Socket-flex-drill"
 			(at 142.24 96.52 0)
 			(effects
