File: pcb/futaba-pcb.kicad_pcb (KiCad board)
At the start: 2 copper layers, 317.2 x 109.9 mm, 106 parts, among them J1 Conn_01x06, SW1 SW_Push, SW10 SW_Push, SW11 SW_Push, SW12 SW_Push, SW13 SW_Push, SW14 SW_Push, SW15 SW_Push, SW16 SW_Push, SW17 SW_Push, SW18 SW_Push, SW2 SW_Push, SW20 SW_Push, SW21 SW_Push, SW22 SW_Push, SW23 SW_Push, SW24 SW_Push, SW25 SW_Push, SW26 SW_Push, SW27 SW_Push, SW28 SW_Push, SW29 SW_Push, SW3 SW_Push, SW30 SW_Push, SW31 SW_Push, SW32 SW_Push, SW33 SW_Push, SW34 SW_Push, SW35 SW_Push, SW36 SW_Push, SW37 SW_Push, SW38 SW_Push, SW39 SW_Push, SW4 SW_Push, SW40 SW_Push, SW41 SW_Push, SW42 SW_Push, SW44 SW_Push, SW45 SW_Push, SW46 SW_Push, SW47 SW_Push, SW48 SW_Push, SW49 SW_Push, SW5 SW_Push, SW50 SW_Push, SW51 SW_Push, SW6 SW_Push, SW7 SW_Push, SW8 SW_Push, SW9 SW_Push, U1 RP2040-Zero

Commit message: Update pcb outline.
Parts:
- moved D5 0.37 mm to (262.4, 91.1)
- moved SW17 0.37 mm to (256.4, 126.0)
- moved Clicker 0.37 mm to (228.8, 152.0)
- moved D45 0.37 mm to (88.6, 144.4)
- moved D22 0.37 mm to (272.7, 156.2)
- moved D24 0.37 mm to (231.8, 168.1)
- moved SW18 0.37 mm to (237.9, 132.0)
- moved SW36 0.37 mm to (139.8, 111.1)
- moved J1 0.37 mm to (216.7, 135.6)
- moved SW35 0.37 mm to (121.3, 105.1)
- moved D7 0.37 mm to (341.6, 115.9)
- moved D34 0.37 mm to (112.2, 101.5)
- moved EC12 0.37 mm to (199.9, 171.5)
- moved SW11 0.37 mm to (254.4, 107.1)
- moved SW28 0.37 mm to (105.2, 77.3)
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Other:
- outline, holes or cut-outs redrawn

Commit message: Update futaba-pcb.kicad_pcb
Other:
- board text added: "Back side"
- board text added: "Front side"
- board text added: "Futaba"
- board text removed: "futaba"
Changed lines of the file:
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@@
 		(fp_arc
 			(start 11.75 11.925002)
-			(mid 12.113834 11.220221)
+			(mid 12.113828 11.220214)
 			(end 12.85 10.925)
 			(stroke
@@
 		(tags "SOD-123")
 		(property "Reference" "D49"
-			(at 0.000001 -2.000003 360)
+			(at 0.000001 -2.000003 0)
 			(layer "F.SilkS")
 			(effects
@@
 		)
 		(property "Value" "1N4148W"
-			(at -0.000001 2.100003 360)
+			(at -0.000001 2.100003 0)
 			(layer "F.Fab")
 			(effects
@@
 		)
 		(fp_text user "${REFERENCE}"
-			(at 0.000001 -2.000003 360)
+			(at 0.000001 -2.000003 0)
 			(layer "F.Fab")
 			(effects
@@
 		(fp_arc
 			(start 11.75 11.925)
-			(mid 12.113824 11.220209)
+			(mid 12.113828 11.220213)
 			(end 12.850001 10.925001)
 			(stroke
@@
 		(at 206.826988 83.677384)
 		(property "Reference" "SW49"
-			(at 14.599999 1.499998 360)
+			(at 14.599999 1.499998 0)
 			(layer "F.SilkS")
 			(effects
@@
 		)
 		(property "Value" "SW_Push"
-			(at 8 1.05 360)
+			(at 8 1.05 0)
 			(layer "F.Fab")
 			(hide yes)
@@
 		(fp_arc
 			(start 11.674999 16.750001)
-			(mid 12.038241 15.902637)
+			(mid 12.038238 15.90263)
 			(end 12.899998 15.574997)
 			(stroke
@@
 		(at 168.826989 83.67738)
 		(property "Reference" "SW51"
-			(at 14.599999 1.499998 360)
+			(at 14.599999 1.499998 0)
 			(layer "F.SilkS")
 			(effects
@@
 		)
 		(property "Value" "SW_Push"
-			(at 8 1.05 360)
+			(at 8 1.05 0)
 			(layer "F.Fab")
 			(hide yes)
@@
 		(fp_arc
 			(start 11.674999 16.750001)
-			(mid 12.038241 15.902637)
+			(mid 12.038238 15.90263)
 			(end 12.899998 15.574997)
 			(stroke
@@
 		(tags "SOD-123")
 		(property "Reference" "D51"
-			(at 0.000001 -2.000003 360)
+			(at 0.000001 -2.000003 0)
 			(layer "F.SilkS")
 			(effects
@@
 		)
 		(property "Value" "1N4148W"
-			(at -0.000001 2.100003 360)
+			(at -0.000001 2.100003 0)
 			(layer "F.Fab")
 			(effects
@@
 		)
 		(fp_text user "${REFERENCE}"
-			(at 0.000001 -2.000003 360)
+			(at 0.000001 -2.000003 0)
 			(layer "F.Fab")
 			(effects
@@
 		)
 		(property "Footprint" "keyboard:RP2040-Zero"
-			(at 0 0 360)
+			(at 0 0 0)
 			(layer "F.Fab")
 			(hide yes)
@@
 		)
 		(property "Datasheet" "https://www.waveshare.com/wiki/RP2040-Zero"
-			(at 0 0 360)
+			(at 0 0 0)
 			(layer "F.Fab")
 			(hide yes)
@@
 		)
 		(property "Description" ""
-			(at 0 0 360)
+			(at 0 0 0)
 			(layer "F.Fab")
 			(hide yes)
@@
 		(tags "SOD-123")
 		(property "Reference" "D50"
-			(at 0.000001 -2.000003 360)
+			(at 0.000001 -2.000003 0)
 			(layer "F.SilkS")
 			(effects
@@
 		)
 		(property "Value" "1N4148W"
-			(at -0.000001 2.100003 360)
+			(at -0.000001 2.100003 0)
 			(layer "F.Fab")
 			(effects
@@
 		)
 		(fp_text user "${REFERENCE}"
-			(at 0.000001 -2.000003 360)
+			(at 0.000001 -2.000003 0)
 			(layer "F.Fab")
 			(effects
@@
 		(tags "connector jushuo horizontal")
 		(property "Reference" "J1"
-			(at 6.02 -2.81 360)
+			(at 6.02 -2.81 0)
 			(layer "F.SilkS")
 			(effects
@@
 		)
 		(property "Value" "Conn_01x06"
-			(at 0.869999 0.11 360)
+			(at 0.869999 0.11 0)
 			(layer "F.Fab")
 			(effects
@@
 		(tags "mounting hole 3.2mm m3 iso14580")
 		(property "Reference" "Clicker"
-			(at 0 -3.75 360)
-			(layer "F.SilkS")
+			(at -0.043536 -4.150433 -0)
+			(layer "B.SilkS")
 			(effects
 				(font
@@
 					(thickness 0.15)
 				)
+				(justify mirror)
 			)
 		)
 		(property "Value" "MountingHole_3.2mm_M3_ISO14580_Pad_TopBottom"
-			(at 0 3.75 360)
+			(at 0 3.75 0)
 			(layer "F.Fab")
 			(effects
@@
 		)
 		(fp_text user "${REFERENCE}"
-			(at 0 0 360)
+			(at 0 0 0)
 			(layer "F.Fab")
 			(effects
@@
 		(tags "SOD-123")
 		(property "Reference" "D19"
-			(at 0.000001 -2.000003 360)
+			(at 0.000001 -2.000003 0)
 			(layer "F.SilkS")
 			(effects
@@
 		)
 		(property "Value" "1N4148W"
-			(at -0.000001 2.100003 360)
+			(at -0.000001 2.100003 0)
 			(layer "F.Fab")
 			(effects
@@
 		)
 		(fp_text user "${REFERENCE}"
-			(at 0.000001 -2.000003 360)
+			(at 0.000001 -2.000003 0)
 			(layer "F.Fab")
 			(effects
@@
 		(at 187.826976 83.677382)
 		(property "Reference" "SW50"
-			(at 14.599999 1.499998 360)
+			(at 14.599999 1.499998 0)
 			(layer "F.SilkS")
 			(effects
@@
 		)
 		(property "Value" "SW_Push"
-			(at 8 1.05 360)
+			(at 8 1.05 0)
 			(layer "F.Fab")
 			(hide yes)
@@
 		(fp_arc
 			(start 11.674999 16.750001)
-			(mid 12.038241 15.902637)
+			(mid 12.038238 15.90263)
 			(end 12.899998 15.574997)
 			(stroke
@@
 		(layer "Edge.Cuts")
 	)
-	(gr_text "futaba"
+	(gr_text "Front side"
+		(at 229.52 133.19 0)
+		(layer "B.SilkS")
+		(effects
+			(font
+				(size 1 1)
+				(thickness 0.15)
+			)
+			(justify left bottom mirror)
+		)
+	)
+	(gr_text "Back side"
+		(at 165.24 133.18 0)
+		(layer "F.SilkS")
+		(effects
+			(font
+				(size 1 1)
+				(thickness 0.15)
+			)
+			(justify left bottom)
+		)
+	)
+	(gr_text "Futaba"
 		(at 164.07133 148.132018 0)
 		(layer "F.SilkS")
@@
 	)
 	(gr_text "rev.1"
-		(at 174.143537 147.873435 0)
+		(at 174.63 148.01 0)
 		(layer "F.SilkS")
 		(effects

Commit message: update pcb
Parts:
- SW22, SW23, SW24, SW46, SW47, SW48: footprint keyboard:Choc_Socket-flex-drill_top -> keyboard:Choc_Socket-flex-drill_mid
Other:
- outline, holes or cut-outs redrawn
- board text added: "rev.2"
- board text removed: "rev.1"
