File: pcb/futaba-pcb.kicad_sch (KiCad schematic)
At the start: 105 parts, among them J1 Conn_01x06, SW1 SW_Push, SW10 SW_Push, SW11 SW_Push, SW12 SW_Push, SW13 SW_Push, SW14 SW_Push, SW15 SW_Push, SW16 SW_Push, SW17 SW_Push, SW18 SW_Push, SW2 SW_Push, SW20 SW_Push, SW21 SW_Push, SW22 SW_Push, SW23 SW_Push, SW24 SW_Push, SW25 SW_Push, SW26 SW_Push, SW27 SW_Push, SW28 SW_Push, SW29 SW_Push, SW3 SW_Push, SW30 SW_Push, SW31 SW_Push, SW32 SW_Push, SW33 SW_Push, SW34 SW_Push, SW35 SW_Push, SW36 SW_Push, SW37 SW_Push, SW38 SW_Push, SW39 SW_Push, SW4 SW_Push, SW40 SW_Push, SW41 SW_Push, SW42 SW_Push, SW44 SW_Push, SW45 SW_Push, SW46 SW_Push, SW47 SW_Push, SW48 SW_Push, SW49 SW_Push, SW5 SW_Push, SW50 SW_Push, SW51 SW_Push, SW6 SW_Push, SW7 SW_Push, SW8 SW_Push, SW9 SW_Push, U1 RP2040-Zero

Commit message: move pcb folder
Parts:
- SW25, SW26, SW27, SW28, SW29, SW30, SW46, SW47, SW48: footprint keyboard:Choc_Socket-flex-drill_2 -> keyboard:Choc_Socket-flex-drill_top
- SW31, SW32, SW33, SW34, SW35, SW36, SW37, SW38, SW39, SW40, SW41: footprint keyboard:Choc_Socket-flex-drill_2 -> keyboard:Choc_Socket-flex-drill
- SW42, SW44, SW45: footprint keyboard:Choc_Socket-flex-drill_2 -> keyboard:Choc_Socket-flex-drill_bottom
- SW49, SW50, SW51: footprint keyboard:Choc_Socket -> keyboard:Choc_Socket-flex-drill_top
Connections:
- net C1: now also U1.4 (GP4); no longer U1.6 (GP6)
- net C2: now also U1.1 (GP1); no longer U1.7 (GP7)
- net C3: now also U1.0 (GP0); no longer U1.5 (GP5)
- net C4: now also U1.7 (GP7); no longer U1.0 (GP0)
- net C5: now also U1.6 (GP6); no longer U1.1 (GP1)
- net C6: now also U1.5 (GP5); no longer U1.4 (GP4)
Other:
- note removed: "Daughter board"
Changed lines of the file:
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@@
 		)
 	)
-	(rectangle
-		(start 251.46 152.4)
-		(end 304.8 190.5)
-		(stroke
-			(width 0)
-			(type default)
-		)
-		(fill
-			(type none)
-		)
-	)
-	(text "Daughter board"
-		(exclude_from_sim no)
-		(at 260.096 154.94 0)
-		(effects
-			(font
-				(size 1.27 1.27)
-			)
-		)
-	)
 	(label "LR2"
 		(at 275.59 82.55 0)
@@
 	)
 	(label "C4"
-		(at 275.59 62.23 0)
+		(at 275.59 80.01 0)
 		(fields_autoplaced yes)
 		(effects
@@
 	)
 	(label "C2"
-		(at 275.59 80.01 0)
+		(at 275.59 64.77 0)
 		(fields_autoplaced yes)
 		(effects
@@
 	)
 	(label "C1"
-		(at 275.59 77.47 0)
+		(at 275.59 72.39 0)
 		(fields_autoplaced yes)
 		(effects
@@
 	)
 	(label "C5"
-		(at 275.59 64.77 0)
+		(at 275.59 77.47 0)
 		(fields_autoplaced yes)
 		(effects
@@
 	)
 	(label "C3"
-		(at 275.59 74.93 0)
+		(at 275.59 62.23 0)
 		(fields_autoplaced yes)
 		(effects
@@
 	)
 	(label "C6"
-		(at 275.59 72.39 0)
+		(at 275.59 74.93 0)
 		(fields_autoplaced yes)
 		(effects
@@
 			)
 		)
-		(property "Footprint" "keyboard:Choc_Socket"
+		(property "Footprint" "keyboard:Choc_Socket-flex-drill_top"
 			(at 69.85 213.36 0)
 			(effects
@@
 			)
 		)
-		(property "Footprint" "keyboard:Choc_Socket-flex-drill_2"
+		(property "Footprint" "keyboard:Choc_Socket-flex-drill_top"
 			(at 118.11 193.04 0)
 			(effects
@@
 			)
 		)
-		(property "Footprint" "keyboard:Choc_Socket-flex-drill_2"
+		(property "Footprint" "keyboard:Choc_Socket-flex-drill_top"
 			(at 93.98 135.89 0)
 			(effects
@@
 			)
 		)
-		(property "Footprint" "keyboard:Choc_Socket-flex-drill_2"
+		(property "Footprint" "keyboard:Choc_Socket-flex-drill"
 			(at 93.98 154.94 0)
 			(effects
@@
 			)
 		)
-		(property "Footprint" "keyboard:Choc_Socket-flex-drill_2"
+		(property "Footprint" "keyboard:Choc_Socket-flex-drill_bottom"
 			(at 166.37 173.99 0)
 			(effects
@@
 			)
 		)
-		(property "Footprint" "keyboard:Choc_Socket-flex-drill_2"
+		(property "Footprint" "keyboard:Choc_Socket-flex-drill_top"
 			(at 142.24 193.04 0)
 			(effects
@@
 			)
 		)
-		(property "Footprint" "keyboard:Choc_Socket-flex-drill_2"
+		(property "Footprint" "keyboard:Choc_Socket-flex-drill"
 			(at 45.72 154.94 0)
 			(effects
@@
 			)
 		)
-		(property "Footprint" "keyboard:Choc_Socket-flex-drill_2"
+		(property "Footprint" "keyboard:Choc_Socket-flex-drill"
 			(at 69.85 173.99 0)
 			(effects
@@
 			)
 		)
-		(property "Footprint" "keyboard:Choc_Socket-flex-drill_2"
+		(property "Footprint" "keyboard:Choc_Socket-flex-drill"
 			(at 45.72 173.99 0)
 			(effects
@@
 			)
 		)
-		(property "Footprint" "keyboard:Choc_Socket-flex-drill_2"
+		(property "Footprint" "keyboard:Choc_Socket-flex-drill_top"
 			(at 142.24 135.89 0)
 			(effects
@@
 			)
 		)
-		(property "Footprint" "keyboard:Choc_Socket-flex-drill_2"
+		(property "Footprint" "keyboard:Choc_Socket-flex-drill"
 			(at 142.24 173.99 0)
 			(effects
@@
 			)
 		)
-		(property "Footprint" "keyboard:Choc_Socket-flex-drill_2"
+		(property "Footprint" "keyboard:Choc_Socket-flex-drill"
 			(at 142.24 154.94 0)
 			(effects
@@
 			)
 		)
-		(property "Footprint" "keyboard:Choc_Socket-flex-drill_2"
+		(property "Footprint" "keyboard:Choc_Socket-flex-drill_top"
 			(at 166.37 193.04 0)
 			(effects
@@
 			)
 		)
-		(property "Footprint" "keyboard:Choc_Socket-flex-drill_2"
+		(property "Footprint" "keyboard:Choc_Socket-flex-drill"
 			(at 166.37 154.94 0)
 			(effects
@@
 			)
 		)
-		(property "Footprint" "keyboard:Choc_Socket-flex-drill_2"
+		(property "Footprint" "keyboard:Choc_Socket-flex-drill_top"
 			(at 69.85 135.89 0)
 			(effects
@@
 			)
 		)
-		(property "Footprint" "keyboard:Choc_Socket-flex-drill_2"
+		(property "Footprint" "keyboard:Choc_Socket-flex-drill"
 			(at 118.11 173.99 0)
 			(effects
@@
 			)
 		)
-		(property "Footprint" "keyboard:Choc_Socket-flex-drill_2"
+		(property "Footprint" "keyboard:Choc_Socket-flex-drill_top"
 			(at 45.72 135.89 0)
 			(effects
@@
 			)
 		)
-		(property "Footprint" "keyboard:Choc_Socket-flex-drill_2"
+		(property "Footprint" "keyboard:Choc_Socket-flex-drill"
 			(at 118.11 154.94 0)
 			(effects
@@
 			)
 		)
-		(property "Footprint" "keyboard:Choc_Socket-flex-drill_2"
+		(property "Footprint" "keyboard:Choc_Socket-flex-drill"
 			(at 69.85 154.94 0)
 			(effects
@@
 			)
 		)
-		(property "Footprint" "keyboard:Choc_Socket-flex-drill_2"
+		(property "Footprint" "keyboard:Choc_Socket-flex-drill"
 			(at 93.98 173.99 0)
 			(effects
@@
 			)
 		)
-		(property "Footprint" "keyboard:Choc_Socket"
+		(property "Footprint" "keyboard:Choc_Socket-flex-drill_top"
 			(at 45.72 213.36 0)
 			(effects
@@
 			)
 		)
-		(property "Footprint" "keyboard:Choc_Socket-flex-drill_2"
+		(property "Footprint" "keyboard:Choc_Socket-flex-drill_bottom"
 			(at 69.85 193.04 0)
 			(effects
@@
 			)
 		)
-		(property "Footprint" "keyboard:Choc_Socket"
+		(property "Footprint" "keyboard:Choc_Socket-flex-drill_top"
 			(at 93.98 213.36 0)
 			(effects
@@
 			)
 		)
-		(property "Footprint" "keyboard:Choc_Socket-flex-drill_2"
+		(property "Footprint" "keyboard:Choc_Socket-flex-drill_top"
 			(at 166.37 135.89 0)
 			(effects
@@
 			)
 		)
-		(property "Footprint" "keyboard:Choc_Socket-flex-drill_2"
+		(property "Footprint" "keyboard:Choc_Socket-flex-drill_bottom"
 			(at 93.98 193.04 0)
 			(effects
@@
 			)
 		)
-		(property "Footprint" "keyboard:Choc_Socket-flex-drill_2"
+		(property "Footprint" "keyboard:Choc_Socket-flex-drill_top"
 			(at 118.11 135.89 0)
 			(effects

Commit message: update pcb
Parts:
- SW22, SW23, SW24, SW46, SW47, SW48: footprint keyboard:Choc_Socket-flex-drill_top -> keyboard:Choc_Socket-flex-drill_mid
Changed lines of the file:
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@@
 			)
 		)
-		(property "Footprint" "keyboard:Choc_Socket-flex-drill_top"
+		(property "Footprint" "keyboard:Choc_Socket-flex-drill_mid"
 			(at 166.37 116.84 0)
 			(effects
@@
 			)
 		)
-		(property "Footprint" "keyboard:Choc_Socket-flex-drill_top"
+		(property "Footprint" "keyboard:Choc_Socket-flex-drill_mid"
 			(at 118.11 193.04 0)
 			(effects
@@
 			)
 		)
-		(property "Footprint" "keyboard:Choc_Socket-flex-drill_top"
+		(property "Footprint" "keyboard:Choc_Socket-flex-drill_mid"
 			(at 142.24 193.04 0)
 			(effects
@@
 			)
 		)
-		(property "Footprint" "keyboard:Choc_Socket-flex-drill_top"
+		(property "Footprint" "keyboard:Choc_Socket-flex-drill_mid"
 			(at 166.37 193.04 0)
 			(effects
@@
 			)
 		)
-		(property "Footprint" "keyboard:Choc_Socket-flex-drill_top"
+		(property "Footprint" "keyboard:Choc_Socket-flex-drill_mid"
 			(at 142.24 116.84 0)
 			(effects
@@
 			)
 		)
-		(property "Footprint" "keyboard:Choc_Socket-flex-drill_top"
+		(property "Footprint" "keyboard:Choc_Socket-flex-drill_mid"
 			(at 118.11 116.84 0)
 			(effects
